Commit message: Update June 2026 capstone source and project documentation

File: src/hospital_robot_description/urdf/robot.urdf.xacro (robot description, xacro)
@@ -1,36 +1,33 @@
 <?xml version="1.0"?>
 <robot xmlns:xacro="http://www.ros.org/wiki/xacro" name="hospital_robot">
-  <!-- ═══════════════════════════════════ -->
-  <!--  파라미터                            -->
-  <!-- ═══════════════════════════════════ -->
-  <xacro:property name="base_radius" value="0.18"/>
-  <xacro:property name="base_height" value="0.12"/>
+  <!-- 휠 -->
+  <xacro:property name="wheel_radius" value="0.0325"/>
+  <xacro:property name="wheel_width" value="0.018"/>
+  <xacro:property name="wheel_separation" value="0.171"/>
+  <xacro:property name="wheel_mass" value="0.5"/>
+  <!-- 차체 (사각형으로 변경) -->
+  <xacro:property name="base_length" value="0.285"/>   <!-- X축 (앞뒤) -->
+  <xacro:property name="base_width" value="0.280"/>    <!-- Y축 (좌우) -->
+  <xacro:property name="base_height" value="0.242"/>   <!-- Z축 (높이) -->
   <xacro:property name="base_mass" value="8.0"/>
-  <xacro:property name="wheel_radius" value="0.05"/>
-  <xacro:property name="wheel_width" value="0.03"/>
-  <xacro:property name="wheel_mass" value="0.5"/>
-  <xacro:property name="wheel_separation" value="0.30"/>
+  <!-- 센서 위치 -->
+  <xacro:property name="lidar_x_offset" value="0.10"/>
+  <xacro:property name="lidar_z_ground" value="0.101"/>   <!-- 10.1cm -->
+  <xacro:property name="camera_x_offset" value="0.152"/>
+  <xacro:property name="camera_z_ground" value="0.056"/>
+  <!-- 기타 -->
   <xacro:property name="caster_radius" value="0.025"/>
   <xacro:property name="caster_mass" value="0.2"/>
   <xacro:property name="lidar_size" value="0.06"/>
   <xacro:property name="lidar_height" value="0.04"/>
-  <xacro:property name="lidar_mass" value="0.3"/>
   <xacro:property name="camera_size" value="0.03"/>
-  <xacro:property name="camera_mass" value="0.1"/>
-  <!-- 색상 -->
   <material name="white"><color rgba="0.95 0.95 0.95 1"/></material>
   <material name="dark_grey"><color rgba="0.3 0.3 0.3 1"/></material>
-  <material name="blue"><color rgba="0.2 0.4 0.8 1"/></material>
+  <material name="black"><color rgba="0.1 0.1 0.1 1"/></material>
   <material name="red"><color rgba="0.8 0.2 0.2 1"/></material>
-  <material name="black"><color rgba="0.1 0.1 0.1 1"/></material>
-  <!-- ═══════════════════════════════════ -->
-  <!--  관성 매크로                         -->
-  <!-- ═══════════════════════════════════ -->
   <xacro:macro name="cylinder_inertia" params="m r h">
     <inertial>
       <mass value="${m}"/>
-      <inertia ixx="${(1/12)*m*(3*r*r+h*h)}" ixy="0" ixz="0"
-               iyy="${(1/12)*m*(3*r*r+h*h)}" iyz="0"
-               izz="${(1/2)*m*r*r}"/>
+      <inertia ixx="${(1/12)*m*(3*r*r+h*h)}" ixy="0" ixz="0" iyy="${(1/12)*m*(3*r*r+h*h)}" iyz="0" izz="${(1/2)*m*r*r}"/>
     </inertial>
   </xacro:macro>
@@ -38,7 +35,5 @@
     <inertial>
       <mass value="${m}"/>
-      <inertia ixx="${(2/5)*m*r*r}" ixy="0" ixz="0"
-               iyy="${(2/5)*m*r*r}" iyz="0"
-               izz="${(2/5)*m*r*r}"/>
+      <inertia ixx="${(2/5)*m*r*r}" ixy="0" ixz="0" iyy="${(2/5)*m*r*r}" iyz="0" izz="${(2/5)*m*r*r}"/>
     </inertial>
   </xacro:macro>
@@ -46,12 +41,7 @@
     <inertial>
       <mass value="${m}"/>
-      <inertia ixx="${(1/12)*m*(y*y+z*z)}" ixy="0" ixz="0"
-               iyy="${(1/12)*m*(x*x+z*z)}" iyz="0"
-               izz="${(1/12)*m*(x*x+y*y)}"/>
+      <inertia ixx="${(1/12)*m*(y*y+z*z)}" ixy="0" ixz="0" iyy="${(1/12)*m*(x*x+z*z)}" iyz="0" izz="${(1/12)*m*(x*x+y*y)}"/>
     </inertial>
   </xacro:macro>
-  <!-- ═══════════════════════════════════ -->
-  <!--  base_footprint                     -->
-  <!-- ═══════════════════════════════════ -->
   <link name="base_footprint"/>
   <joint name="base_joint" type="fixed">
@@ -60,65 +50,24 @@
     <origin xyz="0 0 ${wheel_radius + base_height/2}" rpy="0 0 0"/>
   </joint>
-  <!-- ═══════════════════════════════════ -->
-  <!--  base_link                          -->
-  <!-- ═══════════════════════════════════ -->
+  <!-- 차체: 원형 → 사각형 (Box) -->
   <link name="base_link">
-    <xacro:cylinder_inertia m="${base_mass}" r="${base_radius}" h="${base_height}"/>
+    <xacro:box_inertia m="${base_mass}" x="${base_length}" y="${base_width}" z="${base_height}"/>
     <visual>
-      <geometry>
-        <cylinder radius="${base_radius}" length="${base_height}"/>
-      </geometry>
+      <geometry><box size="${base_length} ${base_width} ${base_height}"/></geometry>
       <material name="white"/>
     </visual>
     <collision>
-      <geometry>
-        <cylinder radius="${base_radius}" length="${base_height}"/>
-      </geometry>
+      <geometry><box size="${base_length} ${base_width} ${base_height}"/></geometry>
     </collision>
   </link>
-  <link name="top_plate">
-    <xacro:cylinder_inertia m="0.3" r="${base_radius - 0.02}" h="0.005"/>
-    <visual>
-      <geometry>
-        <cylinder radius="${base_radius - 0.02}" length="0.005"/>
-      </geometry>
-      <material name="blue"/>
-    </visual>
-  </link>
-  <joint name="top_plate_joint" type="fixed">
-    <parent link="base_link"/>
-    <child link="top_plate"/>
-    <origin xyz="0 0 ${base_height/2 + 0.003}" rpy="0 0 0"/>
-  </joint>
-  <link name="front_marker">
-    <xacro:box_inertia m="0.05" x="0.04" y="0.06" z="0.01"/>
-    <visual>
-      <geometry>
-        <box size="0.04 0.06 0.01"/>
-      </geometry>
-      <material name="red"/>
-    </visual>
-  </link>
-  <joint name="front_marker_joint" type="fixed">
-    <parent link="base_link"/>
-    <child link="front_marker"/>
-    <origin xyz="${base_radius - 0.03} 0 ${base_height/2 + 0.006}" rpy="0 0 0"/>
-  </joint>
-  <!-- ═══════════════════════════════════ -->
-  <!--  구동 바퀴                           -->
-  <!-- ═══════════════════════════════════ -->
   <xacro:macro name="drive_wheel" params="prefix y_offset">
     <link name="${prefix}_wheel">
       <xacro:cylinder_inertia m="${wheel_mass}" r="${wheel_radius}" h="${wheel_width}"/>
       <visual>
-        <geometry>
-          <cylinder radius="${wheel_radius}" length="${wheel_width}"/>
-        </geometry>
+        <geometry><cylinder radius="${wheel_radius}" length="${wheel_width}"/></geometry>
         <material name="dark_grey"/>
       </visual>
       <collision>
-        <geometry>
-          <cylinder radius="${wheel_radius}" length="${wheel_width}"/>
-        </geometry>
+        <geometry><cylinder radius="${wheel_radius}" length="${wheel_width}"/></geometry>
       </collision>
     </link>
@@ -133,45 +82,27 @@
   <xacro:drive_wheel prefix="left" y_offset="${wheel_separation/2}"/>
   <xacro:drive_wheel prefix="right" y_offset="${-wheel_separation/2}"/>
-  <!-- ═══════════════════════════════════ -->
-  <!--  캐스터                              -->
-  <!-- ═══════════════════════════════════ -->
-  <xacro:macro name="caster_wheel" params="prefix x_offset">
-    <link name="${prefix}_caster">
-      <xacro:sphere_inertia m="${caster_mass}" r="${caster_radius}"/>
-      <visual>
-        <geometry>
-          <sphere radius="${caster_radius}"/>
-        </geometry>
-        <material name="black"/>
-      </visual>
-      <collision>
-        <geometry>
-          <sphere radius="${caster_radius}"/>
-        </geometry>
-      </collision>
-    </link>
-    <joint name="${prefix}_caster_joint" type="fixed">
-      <parent link="base_link"/>
-      <child link="${prefix}_caster"/>
-      <origin xyz="${x_offset} 0 ${-base_height/2 - caster_radius + wheel_radius - 0.005}" rpy="0 0 0"/>
-    </joint>
-  </xacro:macro>
-  <xacro:caster_wheel prefix="front" x_offset="${base_radius - 0.04}"/>
-  <xacro:caster_wheel prefix="rear" x_offset="${-base_radius + 0.04}"/>
-  <!-- ═══════════════════════════════════ -->
-  <!--  LiDAR                              -->
-  <!-- ═══════════════════════════════════ -->
-  <link name="lidar_link">
-    <xacro:cylinder_inertia m="${lidar_mass}" r="${lidar_size/2}" h="${lidar_height}"/>
+  <link name="front_caster">
+    <xacro:sphere_inertia m="${caster_mass}" r="${caster_radius}"/>
     <visual>
-      <geometry>
-        <cylinder radius="${lidar_size/2}" length="${lidar_height}"/>
-      </geometry>
-      <material name="dark_grey"/>
+      <geometry><sphere radius="${caster_radius}"/></geometry>
+      <material name="black"/>
     </visual>
     <collision>
-      <geometry>
-        <cylinder radius="${lidar_size/2}" length="${lidar_height}"/>
-      </geometry>
+      <geometry><sphere radius="${caster_radius}"/></geometry>
+    </collision>
+  </link>
+  <joint name="front_caster_joint" type="fixed">
+    <parent link="base_link"/>
+    <child link="front_caster"/>
+    <origin xyz="0.13 0 ${-base_height/2 - caster_radius + wheel_radius - 0.005}" rpy="0 0 0"/>
+  </joint>
+  <link name="lidar_link">
+    <xacro:cylinder_inertia m="0.2" r="${lidar_size/2}" h="${lidar_height}"/>
+    <visual>
+      <geometry><cylinder radius="${lidar_size/2}" length="${lidar_height}"/></geometry>
+      <material name="black"/>
+    </visual>
+    <collision>
+      <geometry><cylinder radius="${lidar_size/2}" length="${lidar_height}"/></geometry>
     </collision>
   </link>
@@ -179,21 +110,14 @@
     <parent link="base_link"/>
     <child link="lidar_link"/>
-    <origin xyz="0 0 ${base_height/2 + lidar_height/2 + 0.01}" rpy="0 0 0"/>
+    <origin xyz="${lidar_x_offset} 0 ${lidar_z_ground - (wheel_radius + base_height/2)}" rpy="0 0 3.14159"/>
   </joint>
-  <!-- ═══════════════════════════════════ -->
-  <!--  카메라                              -->
-  <!-- ═══════════════════════════════════ -->
   <link name="camera_link">
-    <xacro:box_inertia m="${camera_mass}" x="${camera_size}" y="${camera_size*1.5}" z="${camera_size}"/>
+    <xacro:box_inertia m="0.1" x="${camera_size}" y="${camera_size*1.5}" z="${camera_size}"/>
     <visual>
-      <geometry>
-        <box size="${camera_size} ${camera_size*1.5} ${camera_size}"/>
-      </geometry>
-      <material name="black"/>
+      <geometry><box size="${camera_size} ${camera_size*1.5} ${camera_size}"/></geometry>
+      <material name="red"/>
     </visual>
     <collision>
-      <geometry>
-        <box size="${camera_size} ${camera_size*1.5} ${camera_size}"/>
-      </geometry>
+      <geometry><box size="${camera_size} ${camera_size*1.5} ${camera_size}"/></geometry>
     </collision>
   </link>
@@ -201,161 +125,16 @@
     <parent link="base_link"/>
     <child link="camera_link"/>
-    <origin xyz="${base_radius - 0.01} 0 ${base_height/2 - 0.01}" rpy="0 0 0"/>
+    <origin xyz="${camera_x_offset} 0 ${camera_z_ground - (wheel_radius + base_height/2)}" rpy="0 0 0"/>
   </joint>
-  <link name="camera_optical_link"/>
-  <joint name="camera_optical_joint" type="fixed">
-    <parent link="camera_link"/>
-    <child link="camera_optical_link"/>
-    <origin xyz="0 0 0" rpy="${-pi/2} 0 ${-pi/2}"/>
+  <link name="imu_link">
+    <inertial>
+      <mass value="0.01"/>
+      <inertia ixx="0.0001" ixy="0" ixz="0" iyy="0.0001" iyz="0" izz="0.0001"/>
+    </inertial>
+  </link>
+  <joint name="imu_joint" type="fixed">
+    <parent link="base_footprint"/>
+    <child link="imu_link"/>
+    <origin xyz="0 0 0" rpy="0 0 0"/>
   </joint>
-  <!-- ═══════════════════════════════════ -->
-  <!--  Gz Sim 플러그인                     -->
-  <!-- ═══════════════════════════════════ -->
-  <!-- Diff Drive -->
-  <gazebo>
-    <plugin filename="gz-sim-diff-drive-system"
-            name="gz::sim::systems::DiffDrive">
-      <left_joint>left_wheel_joint</left_joint>
-      <right_joint>right_wheel_joint</right_joint>
-      <wheel_separation>${wheel_separation}</wheel_separation>
-      <wheel_radius>${wheel_radius}</wheel_radius>
-      <max_linear_acceleration>0.5</max_linear_acceleration>
-      <max_angular_acceleration>1.0</max_angular_acceleration>
-      <max_linear_velocity>0.5</max_linear_velocity>
-      <max_angular_velocity>1.5</max_angular_velocity>
-      <odom_topic>odom</odom_topic>
-      <tf_topic>tf</tf_topic>
-      <frame_id>odom</frame_id>
-      <child_frame_id>base_footprint</child_frame_id>
-      <odom_publish_frequency>30</odom_publish_frequency>
-      <topic>/cmd_vel</topic>
-    </plugin>
-  </gazebo>
-  <!-- Joint State Publisher -->
-  <gazebo>
-    <plugin filename="gz-sim-joint-state-publisher-system"
-            name="gz::sim::systems::JointStatePublisher">
-      <joint_name>left_wheel_joint</joint_name>
-      <joint_name>right_wheel_joint</joint_name>
-      <update_rate>30</update_rate>
-    </plugin>
-  </gazebo>
-  <!-- 2D LiDAR 센서: gpu_lidar + gz_frame_id를 sensor 안에 -->
-  <gazebo reference="lidar_link">
-    <sensor name="lidar" type="gpu_lidar">
-      <always_on>true</always_on>
-      <update_rate>10</update_rate>
-      <visualize>true</visualize>
-      <topic>scan</topic>
-      <lidar>
-        <scan>
-          <horizontal>
-            <samples>360</samples>
-            <resolution>1</resolution>
-            <min_angle>-3.14159</min_angle>
-            <max_angle>3.14159</max_angle>
-          </horizontal>
-        </scan>
-        <range>
-          <min>0.12</min>
-          <max>12.0</max>
-          <resolution>0.01</resolution>
-        </range>
-        <noise>
-          <type>gaussian</type>
-          <mean>0.0</mean>
-          <stddev>0.005</stddev>
-        </noise>
-      </lidar>
-    </sensor>
-  </gazebo>
-  <!-- 카메라 센서 -->
-  <gazebo reference="camera_link">
-    <sensor name="camera" type="camera">
-      <always_on>true</always_on>
-      <update_rate>15</update_rate>
-      <visualize>true</visualize>
-      <topic>camera/image_raw</topic>
-      <camera>
-        <horizontal_fov>1.22</horizontal_fov>
-        <image>
-          <width>640</width>
-          <height>480</height>
-          <format>R8G8B8</format>
-        </image>
-        <clip>
-          <near>0.05</near>
-          <far>15.0</far>
-        </clip>
-        <noise>
-          <type>gaussian</type>
-          <mean>0.0</mean>
-          <stddev>0.005</stddev>
-        </noise>
-      </camera>
-    </sensor>
-  </gazebo>
-  <!-- 색상 및 마찰 -->
-  <gazebo reference="base_link">
-    <material>
-      <ambient>0.95 0.95 0.95 1</ambient>
-      <diffuse>0.95 0.95 0.95 1</diffuse>
-    </material>
-  </gazebo>
-  <gazebo reference="top_plate">
-    <material>
-      <ambient>0.2 0.4 0.8 1</ambient>
-      <diffuse>0.2 0.4 0.8 1</diffuse>
-    </material>
-  </gazebo>
-  <gazebo reference="front_marker">
-    <material>
-      <ambient>0.8 0.2 0.2 1</ambient>
-      <diffuse>0.8 0.2 0.2 1</diffuse>
-    </material>
-  </gazebo>
-  <gazebo reference="left_wheel">
-    <material>
-      <ambient>0.3 0.3 0.3 1</ambient>
-      <diffuse>0.3 0.3 0.3 1</diffuse>
-    </material>
-    <mu1>1.0</mu1>
-    <mu2>1.0</mu2>
-    <kp>1e6</kp>
-    <kd>1.0</kd>
-  </gazebo>
-  <gazebo reference="right_wheel">
-    <material>
-      <ambient>0.3 0.3 0.3 1</ambient>
-      <diffuse>0.3 0.3 0.3 1</diffuse>
-    </material>
-    <mu1>1.0</mu1>
-    <mu2>1.0</mu2>
-    <kp>1e6</kp>
-    <kd>1.0</kd>
-  </gazebo>
-  <gazebo reference="front_caster">
-    <mu1>0.01</mu1>
-    <mu2>0.01</mu2>
-    <kp>1e6</kp>
-    <kd>1.0</kd>
-  </gazebo>
-  <gazebo reference="rear_caster">
-    <mu1>0.01</mu1>
-    <mu2>0.01</mu2>
-    <kp>1e6</kp>
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